File: tomu.sch (KiCad schematic (older format))
At the start: 15 parts, among them P1 USART0, P2 DEBUG, P3 USB-PCB, U1 EFM32HG309

Commit message: Changing.
Parts:
- U1: value EFM32HG309 -> MKL27Z256VFM4; footprint Housings_DFN_QFN:QFN-24-1EP_5x5mm_Pitch0.65mm -> Housings_DFN_QFN:QFN-32-1EP_5x5mm_Pitch0.5mm; symbol EFM32HG309 -> MKL27Z256VFM4
Changed lines of the file:
@@
 $EndComp
 $Comp
-L EFM32HG309 U1
+L MKL27Z256VFM4 U1
 U 1 1 5798B6D7
 P 4400 4175
 F 0 "U1" H 4350 4125 60  0000 C CNN
-F 1 "EFM32HG309" H 5050 4850 39  0000 C CNN
-F 2 "Housings_DFN_QFN:QFN-24-1EP_5x5mm_Pitch0.65mm" H 4400 4175 60  0001 C CNN
+F 1 "MKL27Z256VFM4" H 5050 4850 39  0000 C CNN
+F 2 "Housings_DFN_QFN:QFN-32-1EP_5x5mm_Pitch0.5mm" H 4400 4175 60  0001 C CNN
 F 3 "" H 4400 4175 60  0000 C CNN
 	1    4400 4175

Commit message: Slowly making work...
Parts:
- C2: value 1uF -> 2.2uF
- R3, R4: value 15 -> 33
Connections:
- wire segments 78 -> 73
Other:
- note added: "Cout"
- note added: "RESET_b pin is dedicated. The port is configured as open drain \nand pullup enabled.\n\nDM and DP I/O pads must connect through series resistors \n(approximately 33 Ω each) to the USB connector on the application \nprinted circuit board (PCB)"
- moved on the sheet: C1, C2, C3, P3, R3, R4, U1

Commit message: Lots of small updates.
Parts:
- removed C1: 1uF, Capacitors_SMD:C_0402, symbol C_Small
- added R?: 10k, Resistors_SMD:R_0402, symbol R_Small
- C3: value 47uF -> 4.7uF
Connections:
- wire segments 73 -> 63
- no-connect marks 3 -> 0
Other:
- note added: "Bootloader Config\n-----\n14 - ~NMI~ - Pull low to enable\n\n10 - PTA0 - SWD_CLK\n13 - PTA3 - SWD_DIO\n\n11 - PTA1 - LPUART0_RX\n12 - PTA2 - LPUART0_TX\n\n20 - PTB0 - I2C0_SCL\n21 - PTB1 - I2C0_SDA\n\n25 - PTC4 - ~SPI0_SS\n26 - PTC5 - SPI0_SCK\n27 - PTC6 - SPI0_MOSI\n28 - PTC7 - SPI0_MISO\n-----\n\nADC \n-----\n 1 - PTE0 - CMP0_OUT\n 9 - PTE30 - DAC0_OUT/ADC0_SE23/CMP0_IN4\n\n20 - PTB0 - ADC0_SE8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"
- note removed: "PB8 - US0_RX\nPB7 - US0_TX\n\nPA0 - Timer 0 Capture Compare Channel 0 -- For PWM - LED0 \nPB7 - Timer 1 Capture Compare Channel 0 -- For PWM - LED1\n\nPC0 - ACMP0_CH0 - Capacitive Touch 0\nPC1 - ACMP0_CH1 - Capacitive Touch 1\n\nPC14 - USB_DM\nPC15 - USB_DP\n\nPE12 - ADC0_CH0\nPE13 - ADC0_CH1\n\nPF0 - DBG_SWCLK #0 - BOOT_RX\nPF1 - DBG_SWDIO #0 - BOOT_TX\n\n"
- moved on the sheet: C2, C3, D1, D2, P1, P2, P3, R1, R2, R3, R4, U1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

Commit message: Getting closer to working.
Parts:
- gave numbers to parts that had none: 1
Changed lines of the file:
@@
 $EndComp
 $Comp
-L GND #PWR01
+L GND #PWR8
 U 1 1 5798BA02
 P 5310 3075
-F 0 "#PWR01" H 5310 2825 50  0001 C CNN
+F 0 "#PWR8" H 5310 2825 50  0001 C CNN
 F 1 "GND" H 5310 2925 50  0000 C CNN
 F 2 "" H 5310 3075 50  0000 C CNN
@@
 DBG_SWDIO
 $Comp
-L GND #PWR02
+L GND #PWR2
 U 1 1 5798EEB6
 P 1235 1775
-F 0 "#PWR02" H 1235 1525 50  0001 C CNN
+F 0 "#PWR2" H 1235 1525 50  0001 C CNN
 F 1 "GND" H 1235 1625 50  0000 C CNN
 F 2 "" H 1235 1775 50  0000 C CNN
@@
 $EndComp
 $Comp
-L +3V3 #PWR03
+L +3V3 #PWR7
 U 1 1 5798EF1D
 P 5110 2475
-F 0 "#PWR03" H 5110 2325 50  0001 C CNN
+F 0 "#PWR7" H 5110 2325 50  0001 C CNN
 F 1 "+3V3" H 5110 2615 50  0000 C CNN
 F 2 "" H 5110 2475 50  0000 C CNN
@@
 $EndComp
 $Comp
-L +3V3 #PWR04
+L +3V3 #PWR1
 U 1 1 5798F04E
 P 1235 1375
-F 0 "#PWR04" H 1235 1225 50  0001 C CNN
+F 0 "#PWR1" H 1235 1225 50  0001 C CNN
 F 1 "+3V3" H 1235 1515 50  0000 C CNN
 F 2 "" H 1235 1375 50  0000 C CNN
@@
 $EndComp
 $Comp
-L GND #PWR05
+L GND #PWR4
 U 1 1 5798FD6B
 P 1235 2550
-F 0 "#PWR05" H 1235 2300 50  0001 C CNN
+F 0 "#PWR4" H 1235 2300 50  0001 C CNN
 F 1 "GND" H 1235 2400 50  0000 C CNN
 F 2 "" H 1235 2550 50  0000 C CNN
@@
 $EndComp
 $Comp
-L +3V3 #PWR06
+L +3V3 #PWR3
 U 1 1 5798FD73
 P 1235 2150
-F 0 "#PWR06" H 1235 2000 50  0001 C CNN
+F 0 "#PWR3" H 1235 2000 50  0001 C CNN
 F 1 "+3V3" H 1235 2290 50  0000 C CNN
 F 2 "" H 1235 2150 50  0000 C CNN
@@
 CAP1B
 $Comp
-L +3V3 #PWR07
+L +3V3 #PWR5
 U 1 1 579B6568
 P 1790 5485
-F 0 "#PWR07" H 1790 5335 50  0001 C CNN
+F 0 "#PWR5" H 1790 5335 50  0001 C CNN
 F 1 "+3V3" H 1790 5625 50  0000 C CNN
 F 2 "" H 1790 5485 50  0000 C CNN
@@
 	2060 4475 2935 4475
 $Comp
-L R_Small R?
+L R_Small R5
 U 1 1 57D4D30F
 P 2735 1950
-F 0 "R?" V 2770 2015 50  0000 L CNN
+F 0 "R5" V 2770 2015 50  0000 L CNN
 F 1 "10k" V 2735 1900 39  0000 L CNN
 F 2 "Resistors_SMD:R_0402" H 2735 1950 50  0001 C CNN
@@
 	2635 1950 2570 1950
 $Comp
-L GND #PWR?
+L GND #PWR6
 U 1 1 57D4D53F
 P 2570 1950
-F 0 "#PWR?" H 2570 1700 50  0001 C CNN
+F 0 "#PWR6" H 2570 1700 50  0001 C CNN
 F 1 "GND" V 2575 1822 50  0000 R CNN
 F 2 "" H 2570 1950 50  0000 C CNN

Commit message: Working on the debug header.
Parts:
- removed P1: USART0, Pin_Headers:Pin_Header_Angled_1x04, symbol CONN_01X04
- removed P2: DEBUG, Pin_Headers:Pin_Header_Angled_1x04, symbol CONN_01X04
- added P1: DEBUG, symbol CONN_01X07
Connections:
- net +3V3: now also P1.5 (P5)
- net DBG_SWCLK: now also P1.1 (P1)
- net DBG_SWDIO: now also P1.4 (P4)
- net GND: now also P1.6 (P6)
- net LEU0_RX: now also U1.11 (PTA1/LPUART0_RX), P1.3 (P3); no longer U1.12 (PTA2/LPUART0_TX)
- net LEU0_TX: now also U1.12 (PTA2/LPUART0_TX), P1.2 (P2); no longer U1.11 (PTA1/LPUART0_RX)
- net RESET: now reaches U1.19 (PTA20/~RESET)
- net RESET: now also P1.7 (P7)
Changed lines of the file:
@@
 	0    1    1    0
 $EndComp
-$Comp
-L CONN_01X04 P2
-U 1 1 5798E965
-P 985 1575
-F 0 "P2" H 985 1825 50  0000 C CNN
-F 1 "DEBUG" V 1085 1575 50  0000 C CNN
-F 2 "Pin_Headers:Pin_Header_Angled_1x04" H 985 1575 50  0001 C CNN
-F 3 "" H 985 1575 50  0000 C CNN
-	1    985  1575
-	-1   0    0    1
-$EndComp
-Text Label 1505 1625 0    39   ~ 0
+Text Label 1235 1525 0    39   ~ 0
 DBG_SWCLK
-Text Label 1505 1525 0    39   ~ 0
+Text Label 1235 1825 0    39   ~ 0
 DBG_SWDIO
-$Comp
-L GND #PWR2
-U 1 1 5798EEB6
-P 1235 1775
-F 0 "#PWR2" H 1235 1525 50  0001 C CNN
-F 1 "GND" H 1235 1625 50  0000 C CNN
-F 2 "" H 1235 1775 50  0000 C CNN
-F 3 "" H 1235 1775 50  0000 C CNN
-	1    1235 1775
-	1    0    0    -1
-$EndComp
 $Comp
 L +3V3 #PWR7
@@
 L +3V3 #PWR1
 U 1 1 5798F04E
-P 1235 1375
-F 0 "#PWR1" H 1235 1225 50  0001 C CNN
-F 1 "+3V3" H 1235 1515 50  0000 C CNN
-F 2 "" H 1235 1375 50  0000 C CNN
-F 3 "" H 1235 1375 50  0000 C CNN
-	1    1235 1375
-	1    0    0    -1
+P 1240 1925
+F 0 "#PWR1" H 1240 1775 50  0001 C CNN
+F 1 "+3V3" V 1235 2140 50  0000 C CNN
+F 2 "" H 1240 1925 50  0000 C CNN
+F 3 "" H 1240 1925 50  0000 C CNN
+	1    1240 1925
+	0    1    1    0
 $EndComp
 $Comp
@@
 $EndComp
 $Comp
-L CONN_01X04 P1
-U 1 1 5798FD61
-P 985 2350
-F 0 "P1" H 985 2600 50  0000 C CNN
-F 1 "USART0" V 1085 2350 50  0000 C CNN
-F 2 "Pin_Headers:Pin_Header_Angled_1x04" H 985 2350 50  0001 C CNN
-F 3 "" H 985 2350 50  0000 C CNN
-	1    985  2350
-	-1   0    0    1
-$EndComp
-$Comp
 L GND #PWR4
 U 1 1 5798FD6B
-P 1235 2550
-F 0 "#PWR4" H 1235 2300 50  0001 C CNN
-F 1 "GND" H 1235 2400 50  0000 C CNN
-F 2 "" H 1235 2550 50  0000 C CNN
-F 3 "" H 1235 2550 50  0000 C CNN
-	1    1235 2550
-	1    0    0    -1
-$EndComp
-$Comp
-L +3V3 #PWR3
-U 1 1 5798FD73
-P 1235 2150
-F 0 "#PWR3" H 1235 2000 50  0001 C CNN
-F 1 "+3V3" H 1235 2290 50  0000 C CNN
-F 2 "" H 1235 2150 50  0000 C CNN
-F 3 "" H 1235 2150 50  0000 C CNN
-	1    1235 2150
-	1    0    0    -1
+P 1240 2025
+F 0 "#PWR4" H 1240 1775 50  0001 C CNN
+F 1 "GND" V 1240 1825 50  0000 C CNN
+F 2 "" H 1240 2025 50  0000 C CNN
+F 3 "" H 1240 2025 50  0000 C CNN
+	1    1240 2025
+	0    -1   -1   0
 $EndComp
 $Comp
@@
 Text Label 2560 3775 0    39   ~ 0
 CAP1A
-Text Label 1660 2300 0    39   ~ 0
+Text Label 1235 1625 0    39   ~ 0
 LEU0_TX
-Text Label 1660 2400 0    39   ~ 0
+Text Label 1235 1725 0    39   ~ 0
 LEU0_RX
-Text Label 5660 2715 0    39   ~ 0
-DEC
 Text Label 2515 5410 1    39   ~ 0
 LED1
@@
 $EndComp
 Wire Wire Line
-	4610 2275 5235 2275
+	4610 2275 4860 2275
+Wire Wire Line
+	4860 2275 5235 2275
 Wire Wire Line
 	4860 2525 4610 2525
@@
 Connection ~ 5235 3025
 Wire Wire Line
-	5235 2275 5235 2775
-Wire Wire Line
-	4860 2275 4860 2600
+	5235 2275 5235 2525
+Wire Wire Line
+	5235 2525 5235 2775
+Wire Wire Line
+	4860 2275 4860 2525
+Wire Wire Line
+	4860 2525 4860 2600
 Wire Wire Line
 	4660 2050 4610 2050
@@
 	4610 2150 4660 2150
 Wire Wire Line
-	4610 1950 5455 1950
+	4610 1950 5410 1950
+Wire Wire Line
+	5410 1950 5455 1950
 Wire Wire Line
 	4860 2050 5455 2050
@@
 	5455 2150 4860 2150
 Wire Wire Line
-	4860 3025 6110 3025
+	4860 3025 5235 3025
+Wire Wire Line
+	5235 3025 5310 3025
+Wire Wire Line
+	5310 3025 5455 3025
+Wire Wire Line
+	5455 3025 6110 3025
 Wire Wire Line
 	6110 3025 6110 2850
@@
 	4860 2600 4610 2600
 Wire Wire Line
-	1185 1625 2065 1625
-Wire Wire Line
-	1185 1525 2145 1525
-Wire Wire Line
-	1185 1725 1235 1725
-Wire Wire Line
-	1235 1725 1235 1775
-Wire Wire Line
-	1185 1425 1235 1425
-Wire Wire Line
-	1235 1425 1235 1375
-Wire Wire Line
 	5110 2475 5110 2525
 Wire Wire Line
@@
 	1790 5485 1790 5435
 Wire Wire Line
-	1665 5435 1890 5435
+	1665 5435 1790 5435
+Wire Wire Line
+	1790 5435 1890 5435
 Connection ~ 1790 5435
 Wire Wire Line
@@
 	1665 4835 1665 5035
 Wire Wire Line
-	1185 2500 1235 2500
-Wire Wire Line
-	1235 2500 1235 2550
-Wire Wire Line
-	1185 2200 1235 2200
-Wire Wire Line
-	1235 2200 1235 2150
+	1185 1925 1240 1925
 Wire Wire Line
 	2515 4835 2515 5835
@@
 Wire Wire Line
 	2515 4835 2265 4835
-Wire Wire Line
-	1185 2300 2935 2300
-Wire Wire Line
-	1185 2400 2935 2400
 Wire Wire Line
 	2440 5935 2440 4985
@@
 $EndComp
 Wire Wire Line
-	4860 2725 4860 3025
+	4860 2725 4860 2800
+Wire Wire Line
+	4860 2800 4860 2875
+Wire Wire Line
+	4860 2875 4860 2950
+Wire Wire Line
+	4860 2950 4860 3025
 Wire Wire Line
 	4860 2725 4610 2725
@@
 Connection ~ 4860 2950
 Wire Wire Line
-	2935 2175 2065 2175
-Wire Wire Line
-	2065 2175 2065 1625
-Wire Wire Line
-	2145 1525 2145 2075
-Wire Wire Line
-	2145 2075 2935 2075
+	2065 2175 2935 2175
+Wire Wire Line
+	2065 1525 2065 2175
+Wire Wire Line
+	1590 2075 2935 2075
 Wire Wire Line
 	2010 4375 2935 4375
@@
 	0    1    1    0
 $EndComp
+Wire Wire Line
+	1590 2075 1590 1825
+Wire Wire Line
+	1590 1825 1185 1825
+Wire Wire Line
+	2065 1525 1185 1525
+Wire Wire Line
+	2935 2400 1970 2400
+Wire Wire Line
+	1970 2400 1970 1625
+Wire Wire Line
+	1970 1625 1185 1625
+Wire Wire Line
+	2935 2300 1880 2300
+Wire Wire Line
+	1880 2300 1880 1725
+Wire Wire Line
+	1880 1725 1185 1725
+$Comp
+L CONN_01X07 P1
+U 1 1 5837D54F
+P 985 1825
+F 0 "P1" H 985 2225 50  0000 C CNN
+F 1 "DEBUG" V 1085 1825 50  0000 C CNN
+F 2 "" H 985 1825 50  0000 C CNN
+F 3 "" H 985 1825 50  0000 C CNN
+	1    985  1825
+	-1   0    0    -1
+$EndComp
+Wire Wire Line
+	1185 2025 1240 2025
+Wire Wire Line
+	2935 2525 1590 2525
+Wire Wire Line
+	1590 2525 1590 2125
+Wire Wire Line
+	1590 2125 1185 2125
+Text Label 1235 2125 0    39   ~ 0
+RESET
 $EndSCHEMATC

Commit message: More work...
Parts:
- P1: footprint (none) -> usb-pcb:debug-points-127mm
Connections:
- net CAP0A: now also W1.1; no longer W1.2
- net CAP0B: now also W1.2; no longer W1.1
- net LEU0_RX: now also P1.2 (P2); no longer P1.3 (P3)
- net LEU0_TX: now also P1.3 (P3); no longer P1.2 (P2)
- no-connect marks 0 -> 2
Other:
- note added: "ADC \n-----\n 1 - PTE0 - CMP0_OUT\n 9 - PTE30 - DAC0_OUT/ADC0_SE23/CMP0_IN4\n\n20 - PTB0 - ADC0_SE8\n21 - PTB1 - ADC0_SE9\n22 - PTC1 - ADC0_SE15\n23 - PTC2 - ADC0_SE11\n\n27 - PTC6 - CMP0_IN0\n28 - PTC7 - CMP0_IN1\n\n30 - PTD5 - ADC0_SE6b\n31 - PTD6 - ADC0_SE7b"
- note added: "Pin 17/18 are blocked\nby Pin 19/Reset trace"
Changed lines of the file:
@@
 $EndComp
 $Comp
-L GND #PWR8
+L GND #PWR01
 U 1 1 5798BA02
 P 5310 3075
-F 0 "#PWR8" H 5310 2825 50  0001 C CNN
+F 0 "#PWR01" H 5310 2825 50  0001 C CNN
 F 1 "GND" H 5310 2925 50  0000 C CNN
 F 2 "" H 5310 3075 50  0000 C CNN
@@
 DBG_SWDIO
 $Comp
-L +3V3 #PWR7
+L +3V3 #PWR02
 U 1 1 5798EF1D
 P 5110 2475
-F 0 "#PWR7" H 5110 2325 50  0001 C CNN
+F 0 "#PWR02" H 5110 2325 50  0001 C CNN
 F 1 "+3V3" H 5110 2615 50  0000 C CNN
 F 2 "" H 5110 2475 50  0000 C CNN
@@
 $EndComp
 $Comp
-L +3V3 #PWR1
+L +3V3 #PWR03
 U 1 1 5798F04E
 P 1240 1925
-F 0 "#PWR1" H 1240 1775 50  0001 C CNN
+F 0 "#PWR03" H 1240 1775 50  0001 C CNN
 F 1 "+3V3" V 1235 2140 50  0000 C CNN
 F 2 "" H 1240 1925 50  0000 C CNN
@@
 $EndComp
 $Comp
-L GND #PWR4
+L GND #PWR04
 U 1 1 5798FD6B
 P 1240 2025
-F 0 "#PWR4" H 1240 1775 50  0001 C CNN
+F 0 "#PWR04" H 1240 1775 50  0001 C CNN
 F 1 "GND" V 1240 1825 50  0000 C CNN
 F 2 "" H 1240 2025 50  0000 C CNN
@@
 F 3 "" H 2335 3575 50  0000 C CNN
 	1    2335 3575
-	1    0    0    -1
+	-1   0    0    -1
 $EndComp
 $Comp
@@
 Text Label 2560 3775 0    39   ~ 0
 CAP1A
+Text Label 1235 1725 0    39   ~ 0
+LEU0_TX
 Text Label 1235 1625 0    39   ~ 0
-LEU0_TX
-Text Label 1235 1725 0    39   ~ 0
 LEU0_RX
 Text Label 2515 5410 1    39   ~ 0
@@
 CAP1B
 $Comp
-L +3V3 #PWR5
+L +3V3 #PWR05
 U 1 1 579B6568
 P 1790 5485
-F 0 "#PWR5" H 1790 5335 50  0001 C CNN
+F 0 "#PWR05" H 1790 5335 50  0001 C CNN
 F 1 "+3V3" H 1790 5625 50  0000 C CNN
 F 2 "" H 1790 5485 50  0000 C CNN
@@
 $EndComp
 Wire Wire Line
-	4610 2275 4860 2275
-Wire Wire Line
-	4860 2275 5235 2275
+	4610 2275 5235 2275
 Wire Wire Line
 	4860 2525 4610 2525
@@
 Connection ~ 5235 3025
 Wire Wire Line
-	5235 2275 5235 2525
-Wire Wire Line
-	5235 2525 5235 2775
-Wire Wire Line
-	4860 2275 4860 2525
-Wire Wire Line
-	4860 2525 4860 2600
+	5235 2275 5235 2775
+Wire Wire Line
+	4860 2275 4860 2600
 Wire Wire Line
 	4660 2050 4610 2050
@@
 	4610 2150 4660 2150
 Wire Wire Line
-	4610 1950 5410 1950
-Wire Wire Line
-	5410 1950 5455 1950
+	4610 1950 5455 1950
 Wire Wire Line
 	4860 2050 5455 2050
@@
 	5455 2150 4860 2150
 Wire Wire Line
-	4860 3025 5235 3025
-Wire Wire Line
-	5235 3025 5310 3025
-Wire Wire Line
-	5310 3025 5455 3025
-Wire Wire Line
-	5455 3025 6110 3025
+	4860 3025 6110 3025
 Wire Wire Line
 	6110 3025 6110 2850
@@
 	1790 5485 1790 5435
 Wire Wire Line
-	1665 5435 1790 5435
-Wire Wire Line
-	1790 5435 1890 5435
+	1665 5435 1890 5435
 Connection ~ 1790 5435
 Wire Wire Line
@@
 $EndComp
 Wire Wire Line
-	4860 2725 4860 2800
-Wire Wire Line
-	4860 2800 4860 2875
-Wire Wire Line
-	4860 2875 4860 2950
-Wire Wire Line
-	4860 2950 4860 3025
+	4860 2725 4860 3025
 Wire Wire Line
 	4860 2725 4610 2725
@@
 	2635 1950 2570 1950
 $Comp
-L GND #PWR6
+L GND #PWR06
 U 1 1 57D4D53F
 P 2570 1950
-F 0 "#PWR6" H 2570 1700 50  0001 C CNN
+F 0 "#PWR06" H 2570 1700 50  0001 C CNN
 F 1 "GND" V 2575 1822 50  0000 R CNN
 F 2 "" H 2570 1950 50  0000 C CNN
@@
 	2065 1525 1185 1525
 Wire Wire Line
-	2935 2400 1970 2400
-Wire Wire Line
-	1970 2400 1970 1625
-Wire Wire Line
-	1970 1625 1185 1625
-Wire Wire Line
-	2935 2300 1880 2300
-Wire Wire Line
-	1880 2300 1880 1725
-Wire Wire Line
-	1880 1725 1185 1725
+	2935 2400 1900 2400
+Wire Wire Line
+	1185 1625 1990 1625
+Wire Wire Line
+	2935 2300 1990 2300
+Wire Wire Line
+	1900 1725 1185 1725
 $Comp
 L CONN_01X07 P1
@@
 F 0 "P1" H 985 2225 50  0000 C CNN
 F 1 "DEBUG" V 1085 1825 50  0000 C CNN
-F 2 "" H 985 1825 50  0000 C CNN
+F 2 "usb-pcb:debug-points-127mm" H 985 1825 50  0001 C CNN
 F 3 "" H 985 1825 50  0000 C CNN
 	1    985  1825
@@
 Text Label 1235 2125 0    39   ~ 0
 RESET
+Wire Wire Line
+	1900 2400 1900 1725
+Wire Wire Line
+	1990 2300 1990 1625
+NoConn ~ 2935 3375
+NoConn ~ 2935 3475
+Text Notes 1850 3305 0    60   ~ 0
+Pin 17/18 are blocked\nby Pin 19/Reset trace
+Text Notes 3930 4990 0    60   ~ 0
+ADC \n-----\n 1 - PTE0 - CMP0_OUT\n 9 - PTE30 - DAC0_OUT/ADC0_SE23/CMP0_IN4\n\n20 - PTB0 - ADC0_SE8\n21 - PTB1 - ADC0_SE9\n22 - PTC1 - ADC0_SE15\n23 - PTC2 - ADC0_SE11\n\n27 - PTC6 - CMP0_IN0\n28 - PTC7 - CMP0_IN1\n\n30 - PTD5 - ADC0_SE6b\n31 - PTD6 - ADC0_SE7b
 $EndSCHEMATC
